File: phasedetector2.kicad_pcb (KiCad board)
At the start: 2 copper layers, 100 x 100 mm, 65 parts, among them J1 Conn_Coaxial, J14 Conn_01x04, J2 Conn_Coaxial, J3 Conn_Coaxial, J5 Conn_Coaxial, J7 DIN41612_02x32_AC, U1 SYPD-52, U15 LT3045xMSE, U16 LT3094xMSE, U2 ADA4898-1YRDZ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

Commit message: layout
Parts:
- moved R9 131.4 mm to (112.5, 135.0), turned to 180 degrees
- moved C1 124.9 mm to (115.5, 138.5), turned to 90 degrees
- moved R7 124.0 mm to (124.5, 139.8)
- moved U2 122.6 mm to (122.3, 135.8), turned to 180 degrees
- moved R5 122.4 mm to (128.0, 139.8), turned to 180 degrees
- moved C2 112.7 mm to (124.0, 131.5)
- moved C13 110.8 mm to (117.8, 74.8)
- moved R16 106.9 mm to (147.5, 127.0), turned to -90 degrees
- moved R18 106.0 mm to (145.5, 127.0), turned to 90 degrees
- moved R17 103.7 mm to (149.5, 127.0), turned to 90 degrees
- moved C14 97.9 mm to (140.5, 122.5)
- moved C6 97.5 mm to (128.1, 102.3)
- moved R15 96.7 mm to (145.5, 112.6), turned to 90 degrees
- moved R14 95.7 mm to (147.5, 112.6), turned to -90 degrees
- moved R12 94.9 mm to (149.5, 112.6), turned to -90 degrees
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Connections:
- C2 pad 2: +5V -> -5V
- C9 pad 2: +5V -> -5V
- U2 pad 4: +5V -> -5V
- U8 pad 4: +5V -> -5V
Routing:
- net +5V: track 18.4 -> 259.9 mm, vias 0 -> 10
- net -5V: track 20.0 -> 158.0 mm, vias 0 -> 6
- net Net-(U2-+): track 0.00 -> 30.6 mm
- net PD: track 0.00 -> 24.5 mm
- net Net-(J5-In): track 0.00 -> 18.9 mm
- net OUTA: track 0.00 -> 17.7 mm
- net Net-(R7-Pad1): track 0.00 -> 16.8 mm
- net Net-(U1-DC): track 0.00 -> 13.1 mm
- net GND: track 38.1 -> 48.5 mm, vias 42 -> 124
- net Net-(U1-RF1): track 0.00 -> 10.0 mm
- net Net-(U9-SA): track 0.00 -> 10.0 mm
- net Net-(U9-SB): track 0.00 -> 8.85 mm
- net Net-(J3-In): track 0.00 -> 7.09 mm
- net Net-(U2--): track 0.00 -> 6.92 mm
- net Net-(U8--): track 0.00 -> 6.69 mm
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Other:
- board text added: "+5V"
- board text added: "-5V"
- board text removed: "+12V"
- board text removed: "-12V"
