File: phasedetector2.kicad_sch (KiCad schematic)
At the start: 45 parts, among them J1 Conn_Coaxial, J2 Conn_Coaxial, J3 Conn_Coaxial, J5 Conn_Coaxial, U1 SYPD-52, U2 ADA4898-1YRDZ, U3 ADC-10-1R, U4 BUF602xDBV, U5 BUF602xDBV, U8 ADA4898-1YRDZ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

Commit message: layout
Connections:
- net +5V: no longer C2.2, C9.2, U2.4 (V-), U8.4 (V-)
- net -5V: now also C2.2, C9.2, U2.4 (V-), U8.4 (V-)
Changed lines of the file:
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@@
 		)
 	)
-	(global_label "+5V"
+	(global_label "-5V"
 		(shape input)
 		(at 205.74 99.06 0)
@@
 		)
 	)
-	(global_label "+5V"
+	(global_label "-5V"
 		(shape input)
 		(at 229.87 144.78 0)

Commit message: kicad 10
Parts:
- R12, R15, R17, R18: value 9k -> 158R
- R14: value 9k -> 200R
- R16: value 9k -> 62R
- R2, R3, R5, R7: value 9k -> 1k
Other:
- note added: "TU-Darmstadt-AQP PDH-module: OPA695 input amps ADA4898-2 before LPF, and as output-buffer LT1568 LPF SYPD-1 phase detector"
- note removed: "OPA695 input amps ADA4898-2 before LPF, and as output-buffer LT1568 LPF SYPD-1 phase detector"
